File: pcb/IMU.kicad_sch (KiCad schematic)
At the start: 4 parts

Commit message: Final PCB Design
Parts:
- C22, C23, C24: footprint (none) -> Capacitor_SMD:C_0402_1005Metric
- MT1: footprint ICM-42670-P:XDCR_ICM-42670-P -> Digikey:ICM-42670-P
Changed lines of the file:
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@@
 			)
 		)
-		(property "Footprint" ""
+		(property "Footprint" "Capacitor_SMD:C_0402_1005Metric"
 			(at 135.5852 57.15 0)
 			(effects
@@
 			)
 		)
-		(property "Footprint" ""
+		(property "Footprint" "Capacitor_SMD:C_0402_1005Metric"
 			(at 138.1252 44.45 0)
 			(effects
@@
 			)
 		)
-		(property "Footprint" "ICM-42670-P:XDCR_ICM-42670-P"
+		(property "Footprint" "Digikey:ICM-42670-P"
 			(at 91.948 43.434 0)
 			(effects
@@
 			)
 		)
-		(property "Footprint" ""
+		(property "Footprint" "Capacitor_SMD:C_0402_1005Metric"
 			(at 124.1552 44.45 0)
 			(effects
