File: pcb/eecsc206a.kicad_sch (KiCad schematic)
At the start: 46 parts, among them J1 Conn_01x03, J18 Conn_01x04, J2 Barrel_Jack, P1 USB_C_Plug_USB2.0, SW1 SW_MEC_5G, SW2 SW_MEC_5G, U1 MAX604, U2 MIC29300-5.0WU, U3 RP2040, U4 W25Q128JVS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

Commit message: Final PCB Design
Parts:
- added H1, H2, H3, H4: MountingHole, MountingHole:MountingHole_3mm_Pad_Via, symbol Mechanical:MountingHole
- added TP5: TestPoint, TestPoint:TestPoint_Pad_D2.0mm, symbol Connector:TestPoint
- C1, C10, C11, C12, C13, C14, C15, C16, C17, C18, C19, C2, C20, C21, C3, C6, C7, C8, C9: footprint (none) -> Capacitor_SMD:C_0402_1005Metric
- C4, C5: footprint (none) -> Capacitor_Tantalum_SMD:CP_EIA-3528-12_Kemet-T
- D1, D2: footprint (none) -> Diode_SMD:D_SOD-323F
- J1: footprint (none) -> Connector_PinHeader_2.54mm:PinHeader_1x03_P2.54mm_Vertical
- J18: footprint (none) -> Connector_Wire:SolderWire-0.1sqmm_1x04_P3.6mm_D0.4mm_OD1mm
- J2: footprint (none) -> Connector_BarrelJack:BarrelJack_Wuerth_694106106102_2.0x5.5mm
- P1: footprint (none) -> Connector_USB:USB_C_Receptacle_Molex_105450-0101
- R1, R2, R3, R4, R5, R6: footprint (none) -> Resistor_SMD:R_0402_1005Metric_Pad0.72x0.64mm_HandSolder
- SW1, SW2: footprint (none) -> Button_Switch_SMD:SW_SPST_FSMSM
- TP1, TP2, TP3, TP4: footprint (none) -> TestPoint:TestPoint_Pad_D2.0mm
- U1, U7: footprint (none) -> Package_SO:PowerIntegrations_SO-8
- U2: footprint TO-263-3_MCL -> Digikey:TO-263-3_MCL
- X1: footprint ABM8-272-T3_ABR -> Digikey:ABM8-272-T3_ABR
Connections:
- net +1V1: now also TP5.1
- net GND: now also C10.2, C11.2, C12.2, C13.2, C7.2, C8.2, C9.2
- net USB-: now reaches R3.2, U3.46 (USB_DM)
- net USB+: now reaches R2.2, U3.47 (USB_DP)
- net +3.3V renamed +3V3
