File: pcb/sensor.kicad_sch (KiCad schematic)
At the start: 85 parts, among them J10 Conn_01x02, J11 Conn_01x02, J12 Conn_01x02, J13 Conn_01x02, J14 Conn_01x02, J15 Conn_01x02, J16 Conn_01x02, J17 Conn_01x02, J8 Conn_01x02, J9 Conn_01x02, U10 LM324, U11 LM321, U6 MAX11127xTI, U8 LM324, U9 LM321

Commit message: Final PCB Design
Parts:
- removed R14, R21: 350, symbol Device:R
- removed R25, R46, R47, R53, R54: 1k, symbol Device:R
- removed R49, R56: 350, symbol Device:R_45deg
- removed U10, U8: LM324, symbol Amplifier_Operational:LM324
- added R14, R21, R25, R46, R47, R53, R54: 348, Resistor_SMD:R_0402_1005Metric_Pad0.72x0.64mm_HandSolder, symbol Device:R_45deg
- added R49, R56: 1k, Resistor_SMD:R_0402_1005Metric_Pad0.72x0.64mm_HandSolder, symbol Device:R
- added U10, U12, U13, U14, U15, U16, U17, U8: LM321, Package_TO_SOT_SMD:SOT-23-5, symbol Amplifier_Operational:LM321
- J10, J11, J12, J13, J14, J15, J16, J17, J8, J9: footprint (none) -> Connector_Wire:SolderWire-0.1sqmm_1x02_P3.6mm_D0.4mm_OD1mm
- R12, R13, R19, R20, R26, R42, R55: value 350 -> 348; footprint (none) -> Resistor_SMD:R_0402_1005Metric_Pad0.72x0.64mm_HandSolder
- R15, R16, R17, R22, R23, R24, R33, R34, R35, R36, R37, R38, R39, R40, R44, R45, R48, R51, R58, R67, R68, R69, R70, R71, R72, R73, R74, R78, R79, R80, R81: footprint (none) -> Resistor_SMD:R_0402_1005Metric_Pad0.72x0.64mm_HandSolder
- R18, R52, R59, R60, R61: value 1k -> 5.6k; footprint (none) -> Resistor_SMD:R_0402_1005Metric_Pad0.72x0.64mm_HandSolder
- R27, R28, R29, R30, R31, R32, R41, R62, R63, R64, R65, R66, R75, R76, R77: value 350 -> 10k; footprint (none) -> Resistor_SMD:R_0402_1005Metric_Pad0.72x0.64mm_HandSolder
- R43, R50, R57: value 350 -> 1k; footprint (none) -> Resistor_SMD:R_0402_1005Metric_Pad0.72x0.64mm_HandSolder
Connections:
- net +3V3: now also R42.2, R14.2, R21.2, R25.2, R46.2, R53.2, U10.5 (V+), U12.5 (V+), U13.5 (V+), U14.5 (V+), U15.5 (V+), U16.5 (V+), U17.5 (V+), U8.5 (V+); no longer J10.1 (Pin_1), J11.1 (Pin_1), J12.1 (Pin_1), J8.1 (Pin_1), J9.1 (Pin_1), R26.2
- net G1: now also U16.4
- net G2: now also R61.2, U8.4
- net G3: now also R60.2, U9.4
- net G4: now also R52.2, U15.4
- net G5: now also R59.2, U6.9 (AIN11), U17.4; no longer R61.2, U6.2 (AIN4), U9.4
- net GND: now also J10.2 (Pin_2), J11.2 (Pin_2), J12.2 (Pin_2), J8.2 (Pin_2), J9.2 (Pin_2), R26.2, R45.2, R51.2, R58.2, R47.2, R54.2, U10.2 (V-), U12.2 (V-), U13.2 (V-), U14.2 (V-), U15.2 (V-), U16.2 (V-), U17.2 (V-), U8.2 (V-); no longer R42.2, R43.2, R50.2, R57.2, R60.2
- net P1: now also U10.4
- net P2: now also U12.4
- net P3: now also U14.4
- net P4: now also U13.4
- net P5: now also U6.10 (AIN12); no longer U6.7 (AIN9)
- net at R17.2, R18.1: now also U16.3 (-)
- net at R23.1: now also R19.1, R20.1; no longer J9.2 (Pin_2)
- net at R17.1: now also R12.1, R13.1; no longer J8.2 (Pin_2)
- net at R60.1, U9.3 (-): now also R44.2; no longer R58.2
- net at R23.2: now also R61.1, U8.3 (-)
- net at R79.2, R81.1: now also U11.3 (-); no longer U11.1 (+)
- net at R33.2, R36.1: now also U12.1 (+)
- net at R35.2, R39.1: now also U12.3 (-)
- net at R67.2, R70.1: now also U13.1 (+)
- net at R26.1, R44.1: now also R25.1; no longer R42.1
- net at R34.2, R38.1: now also U10.1 (+)
- net at R15.1, R16.2: now also U16.1 (+)
- net at R37.2, R40.1: now also U10.3 (-)
- net at R51.1: now also R49.2, U15.1 (+); no longer R48.1
- net at R22.2, R24.1: now also U8.1 (+)
- net at R69.2, R73.1: now also U13.3 (-)
- net at R68.2, R72.1: now also U14.1 (+)
- net at R55.1: now also J12.1 (Pin_1), R56.1; no longer R58.1
- net at R71.2, R74.1: now also U14.3 (-)
- net at R78.2, R80.1: now also U11.1 (+); no longer U11.3 (-)
- new net: J8.1 (Pin_1), R14.1, R16.1
- new net: J10.1 (Pin_1), R42.1, R43.1
- new net: R43.2, R45.1, U9.1 (+)
- new net: R50.2, R52.1, U15.3 (-)
- new net: J9.1 (Pin_1), R21.1, R22.1
- new net: J11.1 (Pin_1), R48.1, R49.1
- new net: R56.2, R58.1, U17.1 (+)
- new net: R53.1, R54.1, R57.1
- new net: R57.2, R59.1, U17.3 (-)
- new net: R46.1, R47.1, R50.1
Other:
- moved on the sheet: J8
