File: pcb/eecsc206a.kicad_pcb (KiCad board)
At the start: 4 copper layers, 99.3 x 109 mm, 157 parts, among them J1 Conn_01x03, J10 Conn_01x02, J11 Conn_01x02, J12 Conn_01x02, J13 Conn_01x02, J14 Conn_01x02, J15 Conn_01x02, J16 Conn_01x02, J17 Conn_01x02, J18 Conn_01x04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

Commit message: Made the PCB Manufacturable
Oopsies
Routing:
- net +3V3: track 118.8 -> 116.7 mm, vias 42 -> 41
- net /IMU/INT: track 18.0 -> 18.7 mm
- net GND: track 189.9 -> 189.3 mm
Other:
- board text added: "G1"
- board text added: "P1"
